File: Adafruit DRV8833.sch (EAGLE design)
At the start: 19 parts, among them J1 VMOTORIN, Q1 DMG3415U, U1 DRV8833PWPR

Commit message: neaten up
Other:
- note removed: "(VMOTOR is safe since internal clamping zener on NSLEEP keeps it below 6.5V)"
- note removed: "Add 20K-75K pullup to VMOTOR for default = on?"
Changed lines of the file:
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@@
 <text x="71.12" y="127" size="1.778" layer="97">Sleep has internal pulldown</text>
 <text x="71.12" y="124.46" size="1.778" layer="97">(= disabled by default)</text>
-<text x="71.12" y="137.16" size="1.778" layer="97">Add 20K-75K pullup to VMOTOR for default = on?</text>
-<text x="71.12" y="134.62" size="1.778" layer="97">(VMOTOR is safe since internal clamping zener on NSLEEP keeps it below 6.5V)</text>
 </plain>
 <instances>
